File: breakout_ag1171/breakout_ag1171.kicad_sch (KiCad schematic)
At the start: 28 parts, among them J1 EXT1, J2 EXT2, J3 Barrel_Jack_Switch, J4 6P6C, J5 FTDI, Q1 Q_NPN_BCE, U1 Ag1171

Commit message: Fix wrong audio channel connections
Parts:
- U1: now in the parts list
Connections:
- net ADC: now also C3.1; no longer C4.1
- net DAC: now also C4.1; no longer C3.1
Other:
- moved on the sheet: C3, C4, R2

Commit message: Exclude U1 from BOM
Parts:
- U1: now left out of the parts list
Connections:
- net +3V3: now also C1.2; no longer C1.1
- net ADC: now also C3.2; no longer C3.1
- net GND: now also C1.1; no longer C1.2
- net at TP3.1, U1.10 (V_{out}): now also C3.1; no longer C3.2
Other:
- moved on the sheet: C1, C3
Changed lines of the file:
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@@
 	(symbol
 		(lib_id "Device:C_Small")
-		(at 133.35 87.63 0)
+		(at 133.35 87.63 180)
 		(unit 1)
 		(exclude_from_sim no)
@@
 		(dnp no)
 		(property "Reference" "C1"
-			(at 135.255 86.995 0)
+			(at 137.795 86.995 0)
 			(effects
 				(font
@@
 		)
 		(property "Value" "10u"
-			(at 135.255 88.9 0)
+			(at 139.065 88.9 0)
 			(effects
 				(font
@@
 		(unit 1)
 		(exclude_from_sim no)
-		(in_bom yes)
+		(in_bom no)
 		(on_board yes)
 		(dnp no)
@@
 	(symbol
 		(lib_id "Device:C_Small")
-		(at 160.02 123.19 270)
+		(at 160.02 123.19 90)
 		(mirror x)
 		(unit 1)
@@
 		)
 		(property "Value" "100n"
-			(at 157.48 128.27 90)
-			(effects
-				(font
+			(at 162.56 128.27 90)
+			(effects
+				(font
